File: Motorc_control/MCU.kicad_sch (KiCad schematic)
At the start: 0 parts

Commit message: Started the MCU Schematic
Parts:
- added C1: 10u, symbol Device:C
- added C10, C9: 2u2, symbol Device:C
- added C12, C2, C3, C4, C5, C6, C7, C8: 100n, symbol Device:C
- added C13: 1u, symbol Device:C
- added FB1: FerriteBead, symbol Device:FerriteBead
- added R1: 0R, symbol Device:R
- added SW1: SW_DIP_x01, symbol Switch:SW_DIP_x01
- added U1: STM32F405RGTx, Package_QFP:LQFP-64_10x10mm_P0.5mm, symbol MCU_ST_STM32F4:STM32F405RGTx
Connections:
- new net: C10.1, U1.47 (VCAP_2)
- new net: C12.1, C13.1, FB1.1, U1.13 (VDDA)
- new net: C9.1, U1.31 (VCAP_1)
- new net: R1.2, U1.60 (BOOT0)
- new net +3.3V: C1.1, C2.1, C3.1, C4.1, C5.1, C6.1, C7.1, FB1.2, R1.1, U1.1 (VBAT), U1.19 (VDD), U1.32 (VDD), U1.48 (VDD), U1.64 (VDD)
- new net GND: C1.2, C10.2, C12.2, C13.2, C2.2, C3.2, C4.2, C5.2, C6.2, C7.2, C8.2, C9.2, SW1.1, U1.12 (VSSA), U1.18 (VSS), U1.63 (VSS)
- new net NRST: C8.1, SW1.2, U1.7 (NRST)
Other:
- note added: "100 nf decoupling cap as close as possible to each power pins"
- note added: "MCU"
- note added: "Power supply schemes 2u2"
- note added: "a 0 Ω resistor on BOOT0, meaning BOOT0 = 0V (GND). Main flash memory (normal mode)"
